File: hs3-arduino/hs3-arduino.kicad_sch (KiCad schematic)
At the start: 33 parts, among them J1 Conn_01x02, J1 Serial, J2 USB_C_Receptacle_USB2.0, J4 LED Data, J5 I2C Header, J6 I2C Header, J7 I2C Header, J8 I2C Header, P1 Power, P2 Analog, P3 Digital, P4 Digital, P5 CONN_01X01, P6 CONN_01X01, P7 CONN_01X01, P8 CONN_01X01, SW1 Reset, SW2 Boot Option, U1 AMS1117-3.3, U2 ESP32-WROOM-32E, U3 TXB0102DCT

Commit message: Adding duplicated Arduino pins
Parts:
- removed R2: 0, symbol Device:R
- removed R5: 10k, Resistor_SMD:R_1206_3216Metric, symbol Device:R
- removed U3: TXB0102DCT, Package_SO:TSSOP-8_3x3mm_P0.65mm, symbol Logic_LevelTranslator:TXB0102DCT
- added P3: Power, Connector_PinHeader_2.54mm:PinHeader_1x08_P2.54mm_Vertical, symbol Connector_Generic:Conn_01x08
- added P4: Analog, Connector_PinHeader_2.54mm:PinHeader_1x06_P2.54mm_Vertical, symbol Connector_Generic:Conn_01x06
- added P7: Digital, Connector_PinHeader_2.54mm:PinHeader_1x10_P2.54mm_Vertical, symbol Connector_Generic:Conn_01x10
- added P8: Digital, Connector_PinHeader_2.54mm:PinHeader_1x08_P2.54mm_Vertical, symbol Connector_Generic:Conn_01x08
- added U?: CH330N, Package_SO:SOIC-8_3.9x4.9mm_P1.27mm, symbol Interface_USB:CH330N
- J5, J6, J7, J8: footprint Connector_JST:JST_XH_B4B-XH-AM_1x04_P2.50mm_Vertical -> Connector_JST:JST_PH_B4B-PH-K_1x04_P2.00mm_Vertical
- renumbered SW2 to BOOT1, J1 to J3, P6 to P10, P7 to P11, P8 to P12, P3 to P5, P4 to P6, P5 to P9, R3 to R2, R4 to R3, SW1 to RST1
Connections:
- net +3V3: now also P3.4 (Pin_4)
- net +5V: now also U1.3 (VI), P3.5 (Pin_5), P3.8 (Pin_8)
- net 0(Rx): now also P8.8 (Pin_8)
- net 1(Tx): now also P8.7 (Pin_7)
- net 10(**/SS): now also P7.8 (Pin_8)
- net 11(**/MOSI): now also P7.7 (Pin_7)
- net 12(MISO): now also P7.6 (Pin_6)
- net 13(SCK): now also P7.5 (Pin_5)
- net 2: now also P8.6 (Pin_6)
- net 3(**): now also P8.5 (Pin_5)
- net 4: now also P8.4 (Pin_4)
- net 5(**): now also P8.3 (Pin_3)
- net 6(**): now also P8.2 (Pin_2)
- net 7: now also P8.1 (Pin_1)
- net 8: now also P7.10 (Pin_10)
- net 9(**): now also P7.9 (Pin_9)
- net A0: now also P4.1 (Pin_1)
- net A1: now also P4.2 (Pin_2)
- net A2: now also P4.3 (Pin_3)
- net A3: now also P4.4 (Pin_4)
- net A4(SDA): now also P4.5 (Pin_5), P7.2 (Pin_2)
- net A5(SCL): now also P4.6 (Pin_6), P7.1 (Pin_1)
- net AREF: now also P7.3 (Pin_3)
- net GND: now also P3.6 (Pin_6), P3.7 (Pin_7), P7.4 (Pin_4)
- net IOREF: now also P3.2 (Pin_2)
- net LED Data: now also J4.1 (Pin_1)
- no-connect marks 20 -> 21
Other:
- note added: "Duplicates of Arduino shield pins"
- moved on the sheet: BOOT1, C1, C2, C3, C4, C5, C6, J1, J2, J3, J4, J5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
