File: hs3-arduino-nano/hs3-arduino-nano.kicad_sch (KiCad schematic)
At the start: 41 parts, among them J1 PWR, J2 USB_B_Micro, J3 DEBUG, J4 I2C, J5 Sensors, J6 ADC, J7 3V3, J8 GND, P1 Digital, P2 Analog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

Commit message: First stab at routing
Parts:
- removed J6: ADC, Connector_PinHeader_2.54mm:PinHeader_1x04_P2.54mm_Vertical, symbol Connector_Generic:Conn_01x04
Changed lines of the file:
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@@
     (pin "1")
-  )
-  (symbol (lib_id "Connector_Generic:Conn_01x04") (at 254.635 180.975 0) (unit 1)
-    (in_bom yes) (on_board yes) (fields_autoplaced)
-    (property "Reference" "J6" (id 0) (at 257.175 180.9749 0)
-      (effects (font (size 1.27 1.27)) (justify left))
-    )
-    (property "Value" "ADC" (id 1) (at 257.175 183.5149 0)
-      (effects (font (size 1.27 1.27)) (justify left))
-    )
-    (property "Footprint" "Connector_PinHeader_2.54mm:PinHeader_1x04_P2.54mm_Vertical" (id 2) (at 254.635 180.975 0)
-      (effects (font (size 1.27 1.27)) hide)
-    )
-    (property "Datasheet" "~" (id 3) (at 254.635 180.975 0)
-      (effects (font (size 1.27 1.27)) hide)
-    )
-    (pin "1")
-    (pin "2")
-    (pin "3")
-    (pin "4")
   )
   (symbol (lib_id "Connector_Generic:Conn_01x05") (at 366.522 88.392 0) (unit 1)
@@
       (reference "J5") (unit 1) (value "Sensors") (footprint "Connector_Hirose:Hirose_DF13-06P-1.25DSA_1x06_P1.25mm_Vertical")
     )
-    (path "/eeb4a81a-6b1d-498e-b4c6-2a8a690418ff"
-      (reference "J6") (unit 1) (value "ADC") (footprint "Connector_PinHeader_2.54mm:PinHeader_1x04_P2.54mm_Vertical")
-    )
     (path "/f19bb86b-894a-4f70-8fd5-97cb3b5bc882"

Commit message: Redone placement, new routing
Parts:
- added ADC: Conn_01x04, Connector_PinHeader_2.00mm:PinHeader_1x04_P2.00mm_Vertical, symbol Connector_Generic:Conn_01x04
- J3: value DEBUG -> DBG
- SW1: value Bootsel -> Boot; footprint Button_Switch_SMD:SW_SPST_B3U-3000P-B -> Button_Switch_SMD:SW_SPST_CK_KXT3
Connections:
- net GPIO26_ADC0: now also ADC.1 (Pin_1)
- net GPIO27_ADC1: now also ADC.2 (Pin_2)
- net GPIO28_ADC2: now also ADC.3 (Pin_3)
- net GPIO29_ADC3: now also ADC.4 (Pin_4)
Changed lines of the file:
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@@
     (in_bom yes) (on_board yes) (fields_autoplaced)
     (property "Reference" "J3" (id 0) (at 147.32 167.64 0))
-    (property "Value" "DEBUG" (id 1) (at 147.32 170.18 0))
+    (property "Value" "DBG" (id 1) (at 147.32 170.18 0))
     (property "Footprint" "Connector_PinHeader_2.54mm:PinHeader_1x02_P2.54mm_Vertical" (id 2) (at 147.32 174.625 0)
       (effects (font (size 1.27 1.27)) hide)
@@
     (pin "1")
     (pin "2")
+  )
+  (symbol (lib_id "Connector_Generic:Conn_01x04") (at 254.635 180.975 0) (unit 1)
+    (in_bom yes) (on_board yes) (fields_autoplaced)
+    (property "Reference" "ADC" (id 0) (at 257.81 180.9749 0)
+      (effects (font (size 1.27 1.27)) (justify left))
+    )
+    (property "Value" "Conn_01x04" (id 1) (at 257.81 183.5149 0)
+      (effects (font (size 1.27 1.27)) (justify left))
+    )
+    (property "Footprint" "Connector_PinHeader_2.00mm:PinHeader_1x04_P2.00mm_Vertical" (id 2) (at 254.635 180.975 0)
+      (effects (font (size 1.27 1.27)) hide)
+    )
+    (property "Datasheet" "~" (id 3) (at 254.635 180.975 0)
+      (effects (font (size 1.27 1.27)) hide)
+    )
+    (pin "1")
+    (pin "2")
+    (pin "3")
+    (pin "4")
   )
   (symbol (lib_id "power:GND") (at 81.915 123.698 0) (unit 1)
@@
       (effects (font (size 1.27 1.27)) (justify right))
     )
-    (property "Value" "Bootsel" (id 1) (at 36.195 117.4749 90)
+    (property "Value" "Boot" (id 1) (at 36.195 117.4749 90)
       (effects (font (size 1.27 1.27)) (justify right))
     )
-    (property "Footprint" "Button_Switch_SMD:SW_SPST_B3U-3000P-B" (id 2) (at 29.845 116.205 0)
+    (property "Footprint" "Button_Switch_SMD:SW_SPST_CK_KXT3" (id 2) (at 29.845 116.205 0)
       (effects (font (size 1.27 1.27)) hide)
     )
@@
       (reference "#PWR029") (unit 1) (value "+3.3V") (footprint "")
     )
+    (path "/1642c8f9-985d-4c88-9e27-ced235e42c18"
+      (reference "ADC") (unit 1) (value "Conn_01x04") (footprint "Connector_PinHeader_2.00mm:PinHeader_1x04_P2.00mm_Vertical")
+    )
     (path "/34a2d67f-22e5-4403-82fa-4be59f69f599"
       (reference "C1") (unit 1) (value "27p") (footprint "Capacitor_SMD:C_0402_1005Metric")
@@
     )
     (path "/120e2590-bb08-4c69-94c5-a585d9315759"
-      (reference "J3") (unit 1) (value "DEBUG") (footprint "Connector_PinHeader_2.54mm:PinHeader_1x02_P2.54mm_Vertical")
+      (reference "J3") (unit 1) (value "DBG") (footprint "Connector_PinHeader_2.54mm:PinHeader_1x02_P2.54mm_Vertical")
     )
     (path "/46799dac-1370-4923-87d2-de884eb986b7"
@@
     )
     (path "/bb6ea6cf-8752-455e-95c0-edab5667069b"
-      (reference "SW1") (unit 1) (value "Bootsel") (footprint "Button_Switch_SMD:SW_SPST_B3U-3000P-B")
+      (reference "SW1") (unit 1) (value "Boot") (footprint "Button_Switch_SMD:SW_SPST_CK_KXT3")
     )
     (path "/90c33843-beb1-4147-99ef-0f56428fc34e"
