File: hs3-arduino-nano/hs3-arduino-nano.kicad_sch (KiCad schematic)
At the start: 42 parts, among them J1 USB_C_Receptacle_USB2.0, J3 DBG, J4 LED, J6 CONN_01x04, J7 CONN_01x04, J8 CONN_01x04, J9 CONN_01x04, P1 Digital, P2 Analog, P3 CONN_01X01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

Commit message: Post-review place & route update pt. 2
Parts:
- renumbered J7 to Sensor1, J8 to Sensor2, J9 to Sensor3
Changed lines of the file:
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@@
   (symbol (lib_id "Connector_Generic:Conn_01x04") (at 337.82 163.195 0) (unit 1)
     (in_bom yes) (on_board yes) (fields_autoplaced)
-    (property "Reference" "J9" (id 0) (at 340.995 163.1949 0)
+    (property "Reference" "Sensor3" (id 0) (at 340.995 163.1949 0)
       (effects (font (size 1.27 1.27)) (justify left))
     )
@@
   (symbol (lib_id "Connector_Generic:Conn_01x04") (at 337.82 151.13 0) (unit 1)
     (in_bom yes) (on_board yes) (fields_autoplaced)
-    (property "Reference" "J8" (id 0) (at 340.995 151.1299 0)
+    (property "Reference" "Sensor2" (id 0) (at 340.995 151.1299 0)
       (effects (font (size 1.27 1.27)) (justify left))
     )
@@
   (symbol (lib_id "Connector_Generic:Conn_01x04") (at 337.82 127 0) (unit 1)
     (in_bom yes) (on_board yes) (fields_autoplaced)
-    (property "Reference" "J6" (id 0) (at 340.995 126.9999 0)
+    (property "Reference" "Sensor0" (id 0) (at 340.995 126.9999 0)
       (effects (font (size 1.27 1.27)) (justify left))
     )
@@
   (symbol (lib_id "Connector_Generic:Conn_01x04") (at 337.82 139.065 0) (unit 1)
     (in_bom yes) (on_board yes) (fields_autoplaced)
-    (property "Reference" "J7" (id 0) (at 340.995 139.0649 0)
+    (property "Reference" "Sensor1" (id 0) (at 340.995 139.0649 0)
       (effects (font (size 1.27 1.27)) (justify left))
     )
@@
       (reference "J4") (unit 1) (value "LED") (footprint "Connector_PinHeader_1.00mm:PinHeader_1x02_P1.00mm_Vertical")
     )
-    (path "/a850f206-7bc0-4e67-91b8-4c9ebd7fa7d6"
-      (reference "J6") (unit 1) (value "CONN_01x04") (footprint "Connector_JST:JST_SH_BM04B-SRSS-TB_1x04-1MP_P1.00mm_Vertical")
-    )
-    (path "/c8efae34-b61b-4d35-894e-88ad84868f4e"
-      (reference "J7") (unit 1) (value "CONN_01x04") (footprint "Connector_JST:JST_SH_BM04B-SRSS-TB_1x04-1MP_P1.00mm_Vertical")
-    )
-    (path "/4b786aef-baa8-422e-baa2-b43ab61ca5de"
-      (reference "J8") (unit 1) (value "CONN_01x04") (footprint "Connector_JST:JST_SH_BM04B-SRSS-TB_1x04-1MP_P1.00mm_Vertical")
-    )
-    (path "/15a603b6-dca3-4476-9025-3b3597941600"
-      (reference "J9") (unit 1) (value "CONN_01x04") (footprint "Connector_JST:JST_SH_BM04B-SRSS-TB_1x04-1MP_P1.00mm_Vertical")
-    )
     (path "/00000000-0000-0000-0000-000056d73fac"
       (reference "P1") (unit 1) (value "Digital") (footprint "Socket_Arduino_Nano:Socket_Strip_Arduino_1x15")
@@
       (reference "SW1") (unit 1) (value "Boot") (footprint "Button_Switch_SMD:SW_SPST_CK_KXT3")
     )
+    (path "/a850f206-7bc0-4e67-91b8-4c9ebd7fa7d6"
+      (reference "Sensor0") (unit 1) (value "CONN_01x04") (footprint "Connector_JST:JST_SH_BM04B-SRSS-TB_1x04-1MP_P1.00mm_Vertical")
+    )
+    (path "/c8efae34-b61b-4d35-894e-88ad84868f4e"
+      (reference "Sensor1") (unit 1) (value "CONN_01x04") (footprint "Connector_JST:JST_SH_BM04B-SRSS-TB_1x04-1MP_P1.00mm_Vertical")
+    )
+    (path "/4b786aef-baa8-422e-baa2-b43ab61ca5de"
+      (reference "Sensor2") (unit 1) (value "CONN_01x04") (footprint "Connector_JST:JST_SH_BM04B-SRSS-TB_1x04-1MP_P1.00mm_Vertical")
+    )
+    (path "/15a603b6-dca3-4476-9025-3b3597941600"
+      (reference "Sensor3") (unit 1) (value "CONN_01x04") (footprint "Connector_JST:JST_SH_BM04B-SRSS-TB_1x04-1MP_P1.00mm_Vertical")
+    )
     (path "/dbeb86be-e9d4-4eaa-9ea6-eae69176406d"

Commit message: Minor cleanup in PCB, adding part numbers to BOM
Parts:
- C1, C2: LCSC (none) -> C1557
- C10, C12, C13, C14, C15, C16, C17, C4, C7, C8: LCSC (none) -> C307331
- C11, C9: LCSC (none) -> C52923
- C3, C5, C6: LCSC (none) -> C15850
- R1: footprint Capacitor_SMD:C_0402_1005Metric -> Resistor_SMD:R_0402_1005Metric; LCSC (none) -> C25905
- R2, R4, R5: LCSC (none) -> C25905
- R3: LCSC (none) -> C25744
- R6, R7: LCSC (none) -> 0402
- SW1: LCSC (none) -> C2689509
- U1: LCSC (none) -> C97521
- U2: LCSC (none) -> C6186
- U3: LCSC (none) -> C2040
- XTAL1: LCSC (none) -> C576558
Changed lines of the file:
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@@
+      (effects (font (size 1.27 1.27)) hide)
+    )
+    (property "LCSC" "C307331" (id 4) (at 173.355 64.135 0)
       (effects (font (size 1.27 1.27)) hide)
     )
@@
     )
     (property "Datasheet" "~" (id 3) (at 161.925 64.135 0)
+      (effects (font (size 1.27 1.27)) hide)
+    )
+    (property "LCSC" "C307331" (id 4) (at 161.925 64.135 0)
       (effects (font (size 1.27 1.27)) hide)
     )
@@
       (effects (font (size 1.27 1.27)) hide)
     )
+    (property "LCSC" "C25905" (id 8) (at 50.8 38.735 0)
+      (effects (font (size 1.27 1.27)) hide)
+    )
     (pin "1")
     (pin "2")
@@
       (effects (font (size 1.27 1.27)) hide)
     )
+    (property "LCSC" "C52923" (id 4) (at 173.355 79.375 0)
+      (effects (font (size 1.27 1.27)) hide)
+    )
     (pin "1")
     (pin "2")
@@
     )
     (property "Datasheet" "~" (id 3) (at 239.395 64.135 0)
+      (effects (font (size 1.27 1.27)) hide)
+    )
+    (property "LCSC" "C307331" (id 4) (at 239.395 64.135 0)
       (effects (font (size 1.27 1.27)) hide)
     )
@@
       (effects (font (size 1.27 1.27)) hide)
     )
+    (property "LCSC" "0402" (id 4) (at 249.555 102.235 0)
+      (effects (font (size 1.27 1.27)) hide)
+    )
     (pin "1")
     (pin "2")
@@
     )
     (property "Datasheet" "~" (id 3) (at 34.925 182.88 0)
+      (effects (font (size 1.27 1.27)) hide)
+    )
+    (property "LCSC" "C1557" (id 4) (at 34.925 182.88 0)
       (effects (font (size 1.27 1.27)) hide)
     )
@@
     )
     (property "Datasheet" "~" (id 3) (at 296.545 64.135 0)
+      (effects (font (size 1.27 1.27)) hide)
+    )
+    (property "LCSC" "C307331" (id 4) (at 296.545 64.135 0)
       (effects (font (size 1.27 1.27)) hide)
     )
@@
       (effects (font (size 1.27 1.27)) hide)
     )
+    (property "LCSC" "C307331" (id 4) (at 78.74 119.38 0)
+      (effects (font (size 1.27 1.27)) hide)
+    )
     (pin "1")
     (pin "2")
@@
     )
     (property "Datasheet" "~" (id 3) (at 78.105 38.735 0)
+      (effects (font (size 1.27 1.27)) hide)
+    )
+    (property "LCSC" "C15850" (id 4) (at 78.105 38.735 0)
       (effects (font (size 1.27 1.27)) hide)
     )
@@
       (effects (font (size 1.27 1.27)) hide)
     )
+    (property "LCSC" "0402" (id 4) (at 249.555 94.615 0)
+      (effects (font (size 1.27 1.27)) hide)
+    )
     (pin "1")
     (pin "2")
@@
     (property "Reference" "R1" (id 0) (at 41.91 133.1722 90))
     (property "Value" "1k" (id 1) (at 41.91 135.4836 90))
-    (property "Footprint" "Capacitor_SMD:C_0402_1005Metric" (id 2) (at 41.91 136.652 90)
+    (property "Footprint" "Resistor_SMD:R_0402_1005Metric" (id 2) (at 41.91 136.652 90)
       (effects (font (size 1.27 1.27)) hide)
     )
@@
       (effects (font (size 1.27 1.27)) hide)
     )
+    (property "LCSC" "C25905" (id 4) (at 41.91 138.43 0)
+      (effects (font (size 1.27 1.27)) hide)
+    )
     (pin "1")
     (pin "2")
@@
     )
     (property "Datasheet" "~" (id 3) (at 57.15 123.19 0)
+      (effects (font (size 1.27 1.27)) hide)
+    )
+    (property "LCSC" "C25744" (id 4) (at 57.15 123.19 0)
       (effects (font (size 1.27 1.27)) hide)
     )
@@
       (effects (font (size 1.27 1.27)) hide)
     )
+    (property "LCSC" "C307331" (id 4) (at 273.685 64.135 0)
+      (effects (font (size 1.27 1.27)) hide)
+    )
     (pin "1")
     (pin "2")
@@
       (effects (font (size 1.27 1.27)) hide)
     )
+    (property "LCSC" "C307331" (id 4) (at 250.825 64.135 0)
+      (effects (font (size 1.27 1.27)) hide)
+    )
     (pin "1")
     (pin "2")
@@
     )
     (property "Datasheet" "~" (id 3) (at 227.965 79.375 0)
+      (effects (font (size 1.27 1.27)) hide)
+    )
+    (property "LCSC" "C52923" (id 4) (at 227.965 79.375 0)
       (effects (font (size 1.27 1.27)) hide)
     )
@@
       (effects (font (size 1.27 1.27)) hide)
     )
+    (property "LCSC" "C25905" (id 8) (at 58.42 41.275 0)
+      (effects (font (size 1.27 1.27)) hide)
+    )
     (pin "1")
     (pin "2")
@@
       (effects (font (size 1.27 1.27)) hide)
     )
+    (property "LCSC" "C25905" (id 4) (at 67.945 193.04 0)
+      (effects (font (size 1.27 1.27)) hide)
+    )
     (pin "1")
     (pin "2")
@@
     )
     (property "Datasheet" "~" (id 3) (at 227.965 64.135 0)
+      (effects (font (size 1.27 1.27)) hide)
+    )
+    (property "LCSC" "C307331" (id 4) (at 227.965 64.135 0)
       (effects (font (size 1.27 1.27)) hide)
     )
@@
     )
     (property "Datasheet" "" (id 3) (at 183.515 142.875 0)
+      (effects (font (size 1.27 1.27)) hide)
+    )
+    (property "LCSC" "C2040" (id 4) (at 202.565 142.875 0)
       (effects (font (size 1.27 1.27)) hide)
     )
@@
       (effects (font (size 1.27 1.27)) hide)
     )
+    (property "LCSC" "C6186" (id 4) (at 95.885 33.655 0)
+      (effects (font (size 1.27 1.27)) hide)
+    )
     (pin "1")
     (pin "2")
@@
     )
     (property "Datasheet" "~" (id 3) (at 262.255 64.135 0)
+      (effects (font (size 1.27 1.27)) hide)
+    )
+    (property "LCSC" "C307331" (id 4) (at 262.255 64.135 0)
       (effects (font (size 1.27 1.27)) hide)
     )
@@
       (effects (font (size 1.524 1.524)))
     )
+    (property "LCSC" "C576558" (id 4) (at 50.8 193.04 0)
+      (effects (font (size 1.27 1.27)) hide)
+    )
     (pin "1")
     (pin "3")
@@
     )
     (property "Datasheet" "~" (id 3) (at 113.665 38.735 0)
+      (effects (font (size 1.27 1.27)) hide)
+    )
+    (property "LCSC" "C15850" (id 4) (at 113.665 38.735 0)
       (effects (font (size 1.27 1.27)) hide)
     )
@@
       (effects (font (size 1.27 1.27)) hide)
     )
+    (property "LCSC" "C2689509" (id 4) (at 25.4 144.907 0)
+      (effects (font (size 1.27 1.27)) hide)
+    )
     (pin "1")
     (pin "2")
@@
     )
     (property "Datasheet" "http://www.winbond.com/resource-files/w25q128jv_dtr%20revc%2003272018%20plus.pdf" (id 3) (at 72.39 140.97 0)
+      (effects (font (size 1.27 1.27)) hide)
+    )
+    (property "LCSC" "C97521" (id 4) (at 72.39 140.97 0)
       (effects (font (size 1.27 1.27)) hide)
     )
@@
       (effects (font (size 1.27 1.27)) hide)
     )
+    (property "LCSC" "C307331" (id 4) (at 285.115 64.135 0)
+      (effects (font (size 1.27 1.27)) hide)
+    )
     (pin "1")
     (pin "2")
@@
     )
     (property "Datasheet" "~" (id 3) (at 34.925 193.04 0)
+      (effects (font (size 1.27 1.27)) hide)
+    )
+    (property "LCSC" "C1557" (id 4) (at 34.925 193.04 0)
       (effects (font (size 1.27 1.27)) hide)
     )
@@
       (effects (font (size 1.27 1.27)) hide)
     )
+    (property "LCSC" "C15850" (id 4) (at 87.63 70.485 0)
+      (effects (font (size 1.27 1.27)) hide)
+    )
     (pin "1")
     (pin "2")
@@
     )
     (path "/5f48140c-abf7-4d9a-98cc-d14aa4e18fee"
-      (reference "R1") (unit 1) (value "1k") (footprint "Capacitor_SMD:C_0402_1005Metric")
+      (reference "R1") (unit 1) (value "1k") (footprint "Resistor_SMD:R_0402_1005Metric")
     )
     (path "/25ce359b-de1e-4737-b3c7-b8d15a1df2cc"

Commit message: Adding manufacturing files
Parts:
- C1, C10, C11, C12, C13, C14, C15, C16, C17, C2, C4, C7, C8, C9, R1, R2, R3, R4, R5, R6, R7: JLC (none) -> 0402
- C3, C5, C6: JLC (none) -> 0805
- SW1: JLC (none) -> SW-SMD
- U1: JLC (none) -> SOIC-8_5.3x5.3x1.27P
- U2: JLC (none) -> SOT-223
- U3: JLC (none) -> LQFN-56_EP_7.0x7.0x0.4P
- XTAL1: JLC (none) -> SMD2016
Changed lines of the file:
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@@
+      (effects (font (size 1.27 1.27)) hide)
+    )
+    (property "JLC" "0402" (id 5) (at 173.355 64.135 0)
       (effects (font (size 1.27 1.27)) hide)
     )
@@
     )
     (property "LCSC" "C307331" (id 4) (at 161.925 64.135 0)
+      (effects (font (size 1.27 1.27)) hide)
+    )
+    (property "JLC" "0402" (id 5) (at 161.925 64.135 0)
       (effects (font (size 1.27 1.27)) hide)
     )
@@
       (effects (font (size 1.27 1.27)) hide)
     )
+    (property "JLC" "0402" (id 9) (at 50.8 38.735 0)
+      (effects (font (size 1.27 1.27)) hide)
+    )
     (pin "1")
     (pin "2")
@@
       (effects (font (size 1.27 1.27)) hide)
     )
+    (property "JLC" "0402" (id 5) (at 173.355 79.375 0)
+      (effects (font (size 1.27 1.27)) hide)
+    )
     (pin "1")
     (pin "2")
@@
     )
     (property "LCSC" "C307331" (id 4) (at 239.395 64.135 0)
+      (effects (font (size 1.27 1.27)) hide)
+    )
+    (property "JLC" "0402" (id 5) (at 239.395 64.135 0)
       (effects (font (size 1.27 1.27)) hide)
     )
@@
       (effects (font (size 1.27 1.27)) hide)
     )
+    (property "JLC" "0402" (id 5) (at 249.555 102.235 0)
+      (effects (font (size 1.27 1.27)) hide)
+    )
     (pin "1")
     (pin "2")
@@
     )
     (property "LCSC" "C1557" (id 4) (at 34.925 182.88 0)
+      (effects (font (size 1.27 1.27)) hide)
+    )
+    (property "JLC" "0402" (id 5) (at 34.925 182.88 0)
       (effects (font (size 1.27 1.27)) hide)
     )
@@
     )
     (property "LCSC" "C307331" (id 4) (at 296.545 64.135 0)
+      (effects (font (size 1.27 1.27)) hide)
+    )
+    (property "JLC" "0402" (id 5) (at 296.545 64.135 0)
       (effects (font (size 1.27 1.27)) hide)
     )
@@
       (effects (font (size 1.27 1.27)) hide)
     )
+    (property "JLC" "0402" (id 5) (at 78.74 119.38 0)
+      (effects (font (size 1.27 1.27)) hide)
+    )
     (pin "1")
     (pin "2")
@@
     )
     (property "LCSC" "C15850" (id 4) (at 78.105 38.735 0)
+      (effects (font (size 1.27 1.27)) hide)
+    )
+    (property "JLC" "0805" (id 5) (at 78.105 38.735 0)
       (effects (font (size 1.27 1.27)) hide)
     )
@@
       (effects (font (size 1.27 1.27)) hide)
     )
+    (property "JLC" "0402" (id 5) (at 249.555 94.615 0)
+      (effects (font (size 1.27 1.27)) hide)
+    )
     (pin "1")
     (pin "2")
@@
       (effects (font (size 1.27 1.27)) hide)
     )
+    (property "JLC" "0402" (id 5) (at 41.91 138.43 0)
+      (effects (font (size 1.27 1.27)) hide)
+    )
     (pin "1")
     (pin "2")
@@
     )
     (property "LCSC" "C25744" (id 4) (at 57.15 123.19 0)
+      (effects (font (size 1.27 1.27)) hide)
+    )
+    (property "JLC" "0402" (id 5) (at 57.15 123.19 0)
       (effects (font (size 1.27 1.27)) hide)
     )
@@
       (effects (font (size 1.27 1.27)) hide)
     )
+    (property "JLC" "0402" (id 5) (at 273.685 64.135 0)
+      (effects (font (size 1.27 1.27)) hide)
+    )
     (pin "1")
     (pin "2")
@@
       (effects (font (size 1.27 1.27)) hide)
     )
+    (property "JLC" "0402" (id 5) (at 250.825 64.135 0)
+      (effects (font (size 1.27 1.27)) hide)
+    )
     (pin "1")
     (pin "2")
@@
     )
     (property "LCSC" "C52923" (id 4) (at 227.965 79.375 0)
+      (effects (font (size 1.27 1.27)) hide)
+    )
+    (property "JLC" "0402" (id 5) (at 227.965 79.375 0)
       (effects (font (size 1.27 1.27)) hide)
     )
@@
       (effects (font (size 1.27 1.27)) hide)
     )
+    (property "JLC" "0402" (id 9) (at 58.42 41.275 0)
+      (effects (font (size 1.27 1.27)) hide)
+    )
     (pin "1")
     (pin "2")
@@
       (effects (font (size 1.27 1.27)) hide)
     )
+    (property "JLC" "0402" (id 5) (at 67.945 193.04 0)
+      (effects (font (size 1.27 1.27)) hide)
+    )
     (pin "1")
     (pin "2")
@@
     )
     (property "LCSC" "C307331" (id 4) (at 227.965 64.135 0)
+      (effects (font (size 1.27 1.27)) hide)
+    )
+    (property "JLC" "0402" (id 5) (at 227.965 64.135 0)
       (effects (font (size 1.27 1.27)) hide)
     )
@@
     )
     (property "LCSC" "C2040" (id 4) (at 202.565 142.875 0)
+      (effects (font (size 1.27 1.27)) hide)
+    )
+    (property "JLC" "LQFN-56_EP_7.0x7.0x0.4P" (id 5) (at 202.565 142.875 0)
       (effects (font (size 1.27 1.27)) hide)
     )
@@
       (effects (font (size 1.27 1.27)) hide)
     )
+    (property "JLC" "SOT-223" (id 5) (at 95.885 33.655 0)
+      (effects (font (size 1.27 1.27)) hide)
+    )
     (pin "1")
     (pin "2")
@@
     )
     (property "LCSC" "C307331" (id 4) (at 262.255 64.135 0)
+      (effects (font (size 1.27 1.27)) hide)
+    )
+    (property "JLC" "0402" (id 5) (at 262.255 64.135 0)
       (effects (font (size 1.27 1.27)) hide)
     )
@@
       (effects (font (size 1.27 1.27)) hide)
     )
+    (property "JLC" "SMD2016" (id 5) (at 50.8 193.04 0)
+      (effects (font (size 1.27 1.27)) hide)
+    )
     (pin "1")
     (pin "3")
@@
     )
     (property "LCSC" "C15850" (id 4) (at 113.665 38.735 0)
+      (effects (font (size 1.27 1.27)) hide)
+    )
+    (property "JLC" "0805" (id 5) (at 113.665 38.735 0)
       (effects (font (size 1.27 1.27)) hide)
     )
@@
       (effects (font (size 1.27 1.27)) hide)
     )
+    (property "JLC" "SW-SMD" (id 5) (at 25.4 144.907 0)
+      (effects (font (size 1.27 1.27)) hide)
+    )
     (pin "1")
     (pin "2")
@@
     )
     (property "LCSC" "C97521" (id 4) (at 72.39 140.97 0)
+      (effects (font (size 1.27 1.27)) hide)
+    )
+    (property "JLC" "SOIC-8_5.3x5.3x1.27P" (id 5) (at 72.39 140.97 0)
       (effects (font (size 1.27 1.27)) hide)
     )
@@
       (effects (font (size 1.27 1.27)) hide)
     )
+    (property "JLC" "0402" (id 5) (at 285.115 64.135 0)
+      (effects (font (size 1.27 1.27)) hide)
+    )
     (pin "1")
     (pin "2")
@@
     )
     (property "LCSC" "C1557" (id 4) (at 34.925 193.04 0)
+      (effects (font (size 1.27 1.27)) hide)
+    )
+    (property "JLC" "0402" (id 5) (at 34.925 193.04 0)
       (effects (font (size 1.27 1.27)) hide)
     )
@@
       (effects (font (size 1.27 1.27)) hide)
     )
+    (property "JLC" "0805" (id 5) (at 87.63 70.485 0)
+      (effects (font (size 1.27 1.27)) hide)
+    )

Commit message: Fixing footprint for xtal
Parts:
- XTAL1: footprint Crystal:Crystal_SMD_3225-4Pin_3.2x2.5mm -> Crystal:Crystal_SMD_2016-4Pin_2.0x1.6mm
Changed lines of the file:
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@@
       (effects (font (size 1.524 1.524)) (justify right))
     )
-    (property "Footprint" "Crystal:Crystal_SMD_3225-4Pin_3.2x2.5mm" (id 2) (at 59.944 187.96 0)
+    (property "Footprint" "Crystal:Crystal_SMD_2016-4Pin_2.0x1.6mm" (id 2) (at 59.944 187.96 0)
       (effects (font (size 1.524 1.524)) hide)
     )
@@
     )
     (path "/b041487f-0668-4406-889e-c637618ffac1"
-      (reference "XTAL1") (unit 1) (value "XRCGB27M120F3M00R0") (footprint "Crystal:Crystal_SMD_3225-4Pin_3.2x2.5mm")
-    )
-  )
+      (reference "XTAL1") (unit 1) (value "XRCGB27M120F3M00R0") (footprint "Crystal:Crystal_SMD_2016-4Pin_2.0x1.6mm")
+    )
+  )

Commit message: Fixing incorrect XTAL1 part number
Parts:
- R5: value 1k -> 0; LCSC C25905 -> C17168
- XTAL1: value XRCGB27M120F3M00R0 -> OT201612MJBA4SL; JLC SMD2016 -> SMD-2016-4P; LCSC C576558 -> C669076
Changed lines of the file:
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@@
     (in_bom yes) (on_board yes)
     (property "Reference" "R5" (id 0) (at 67.945 187.7822 90))
-    (property "Value" "1k" (id 1) (at 67.945 190.0936 90))
+    (property "Value" "0" (id 1) (at 67.945 190.0936 90))
     (property "Footprint" "Resistor_SMD:R_0402_1005Metric" (id 2) (at 67.945 191.262 90)
       (effects (font (size 1.27 1.27)) hide)
@@
       (effects (font (size 1.27 1.27)) hide)
     )
-    (property "LCSC" "C25905" (id 4) (at 67.945 193.04 0)
+    (property "LCSC" "C17168" (id 4) (at 67.945 193.04 0)
       (effects (font (size 1.27 1.27)) hide)
     )
@@
       (effects (font (size 1.524 1.524)) (justify right))
     )
-    (property "Value" "XRCGB27M120F3M00R0" (id 1) (at 37.465 180.34 90)
+    (property "Value" "OT201612MJBA4SL" (id 1) (at 37.465 180.34 90)
       (effects (font (size 1.524 1.524)) (justify right))
     )
@@
       (effects (font (size 1.524 1.524)))
     )
-    (property "LCSC" "C576558" (id 4) (at 50.8 193.04 0)
-      (effects (font (size 1.27 1.27)) hide)
-    )
-    (property "JLC" "SMD2016" (id 5) (at 50.8 193.04 0)
+    (property "LCSC" "C669076" (id 4) (at 50.8 193.04 0)
+      (effects (font (size 1.27 1.27)) hide)
+    )
+    (property "JLC" "SMD-2016-4P" (id 5) (at 50.8 193.04 0)
       (effects (font (size 1.27 1.27)) hide)
     )
@@
     )
     (path "/8ec824ce-929c-437b-8b37-f4317ee34db7"
-      (reference "R5") (unit 1) (value "1k") (footprint "Resistor_SMD:R_0402_1005Metric")
+      (reference "R5") (unit 1) (value "0") (footprint "Resistor_SMD:R_0402_1005Metric")
     )
     (path "/5e6ff893-4137-4ea9-b15c-bf7d80927966"
@@
     )
     (path "/b041487f-0668-4406-889e-c637618ffac1"
-      (reference "XTAL1") (unit 1) (value "XRCGB27M120F3M00R0") (footprint "Crystal:Crystal_SMD_2016-4Pin_2.0x1.6mm")
-    )
-  )
+      (reference "XTAL1") (unit 1) (value "OT201612MJBA4SL") (footprint "Crystal:Crystal_SMD_2016-4Pin_2.0x1.6mm")
+    )
+  )
